File: blaze-radio.kicad_sch (KiCad schematic)
At the start: 5 parts, among them J1 Conn_02x08_Castelated

Commit message: Readability updates
Parts:
- renumbered D2 to D1, D1 to D2, R4 to R1, R1 to R2
Connections:
- net RF_OUT renamed ANTENNA
Other:
- sheet Transceiver ports: added ANTENNA; removed RF_IN
- moved on the sheet: D1, D2, R1, R2

Commit message: Routing updates
Parts:
- D1, D2: footprint LED_SMD:LED_0402_1005Metric -> LED_SMD:LED_0201_0603Metric
- J1: now left out of the parts list
Connections:
- net PD04 is gone; now on net PC00: J1.16 (Pin_16)
- net +3V3: now also D1.2 (A)
- net GND: no longer R1.2
- net PA_nEN: now also R1.2
- net PC00: no longer J1.15 (Pin_15)
- net VDD: no longer D1.2 (A)
- new net PC02: J1.15 (Pin_15)
Other:
- sheet Transceiver ports: added PC02; removed PD04
