File: power-amp.kicad_sch (KiCad schematic)
At the start: 12 parts, among them U3 TSS-13HLN+

Commit message: Readability updates
Parts:
- renumbered C23 to C19, C24 to C20, C25 to C21, C26 to C22, C27 to C23, C28 to C24, C29 to C25, R2 to R3, R3 to R4, U3 to U2
Other:
- moved on the sheet: C20, C24, C25, L7

Commit message: Routing updates
Connections:
- net at C23.1, L7.2: no longer C19.1
- net at C23.2, U2.3 (IN): now also C19.1
Other:
- moved on the sheet: C23, C25, L7
Changed lines of the file:
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@@
 	)
 	(junction
-		(at 81.28 63.5)
+		(at 80.01 63.5)
+		(diameter 0)
+		(color 0 0 0 0)
+	)
+	(junction
+		(at 93.98 63.5)
 		(diameter 0)
 		(color 0 0 0 0)
@@
 	)
 	(junction
-		(at 91.44 63.5)
-		(diameter 0)
-		(color 0 0 0 0)
-	)
-	(junction
 		(at 101.6 57.15)
 		(diameter 0)
@@
 	(wire
 		(pts
-			(xy 91.44 44.45) (xy 91.44 63.5)
+			(xy 93.98 44.45) (xy 93.98 63.5)
 		)
 		(stroke
@@
 	(wire
 		(pts
-			(xy 78.74 63.5) (xy 81.28 63.5)
-		)
-		(stroke
-			(width 0)
-			(type default)
-		)
-	)
-	(wire
-		(pts
-			(xy 95.25 44.45) (xy 91.44 44.45)
+			(xy 77.47 63.5) (xy 80.01 63.5)
 		)
 		(stroke
@@
 	(wire
 		(pts
+			(xy 93.98 44.45) (xy 95.25 44.45)
+		)
+		(stroke
+			(width 0)
+			(type default)
+		)
+	)
+	(wire
+		(pts
 			(xy 102.87 53.34) (xy 101.6 53.34)
 		)
@@
 	(wire
 		(pts
-			(xy 81.28 63.5) (xy 83.82 63.5)
+			(xy 80.01 63.5) (xy 82.55 63.5)
 		)
 		(stroke
@@
 	(wire
 		(pts
+			(xy 87.63 63.5) (xy 88.9 63.5)
+		)
+		(stroke
+			(width 0)
+			(type default)
+		)
+	)
+	(wire
+		(pts
+			(xy 93.98 63.5) (xy 96.52 63.5)
+		)
+		(stroke
+			(width 0)
+			(type default)
+		)
+	)
+	(wire
+		(pts
 			(xy 109.22 53.34) (xy 107.95 53.34)
-		)
-		(stroke
-			(width 0)
-			(type default)
-		)
-	)
-	(wire
-		(pts
-			(xy 88.9 63.5) (xy 91.44 63.5)
 		)
 		(stroke
@@
 	(hierarchical_label "RF_IN"
 		(shape input)
-		(at 78.74 63.5 180)
+		(at 77.47 63.5 180)
 		(effects
 			(font
@@
 	(symbol
 		(lib_id "Device:C_Small")
-		(at 93.98 63.5 90)
+		(at 91.44 63.5 90)
 		(unit 1)
 		(exclude_from_sim no)
@@
 		(dnp no)
 		(property "Reference" "C23"
-			(at 93.9863 57.15 90)
+			(at 91.4463 57.15 90)
 			(effects
 				(font
@@
 		)
 		(property "Value" "2.2uF"
-			(at 95.25 59.69 90)
+			(at 91.186 59.69 90)
 			(effects
 				(font
@@
 		)
 		(property "Footprint" "Capacitor_SMD:C_0402_1005Metric"
-			(at 93.98 63.5 0)
+			(at 91.44 63.5 0)
 			(effects
 				(font
@@
 		)
 		(property "Datasheet" "~"
-			(at 93.98 63.5 0)
+			(at 91.44 63.5 0)
 			(effects
 				(font
@@
 		)
 		(property "Description" "Unpolarized capacitor, small symbol"
-			(at 93.98 63.5 0)
+			(at 91.44 63.5 0)
 			(effects
 				(font
@@
 		)
 		(property "Manufacturer" "Murata"
-			(at 93.98 63.5 90)
+			(at 91.44 63.5 90)
 			(effects
 				(font
@@
 		)
 		(property "Part_Number" "GRM188C71E225KE11D"
-			(at 93.98 63.5 90)
+			(at 91.44 63.5 90)
 			(effects
 				(font
@@
 	(symbol
 		(lib_id "Device:C_Small")
-		(at 81.28 66.04 180)
+		(at 80.01 66.04 180)
 		(unit 1)
 		(exclude_from_sim no)
@@
 		(dnp no)
 		(property "Reference" "C25"
-			(at 74.168 65.786 0)
+			(at 72.898 65.786 0)
 			(effects
 				(font
@@
 		)
 		(property "Value" "1.5pF"
-			(at 74.168 68.326 0)
+			(at 72.898 68.326 0)
 			(effects
 				(font
@@
 		)
 		(property "Footprint" "Capacitor_SMD:C_0201_0603Metric"
-			(at 81.28 66.04 0)
+			(at 80.01 66.04 0)
 			(effects
 				(font
@@
 		)
 		(property "Datasheet" "~"
-			(at 81.28 66.04 0)
+			(at 80.01 66.04 0)
 			(effects
 				(font
@@
 		)
 		(property "Description" "Unpolarized capacitor, small symbol"
-			(at 81.28 66.04 0)
+			(at 80.01 66.04 0)
 			(effects
 				(font
@@
 		)
 		(property "Manufacturer" "Murata"
-			(at 81.28 66.04 0)
+			(at 80.01 66.04 0)
 			(effects
 				(font
@@
 		)
 		(property "Part_Number" "GRM1555C1H1R5CA1D"
-			(at 81.28 66.04 0)
+			(at 80.01 66.04 0)
 			(effects
 				(font
@@
 	(symbol
 		(lib_id "power:GND")
-		(at 81.28 68.58 0)
+		(at 80.01 68.58 0)
 		(unit 1)
 		(exclude_from_sim no)
@@
 		(fields_autoplaced yes)
 		(property "Reference" "#PWR035"
-			(at 81.28 74.93 0)
+			(at 80.01 74.93 0)
 			(effects
 				(font
@@
 		)
 		(property "Value" "GND"
-			(at 81.28 73.66 0)
+			(at 80.01 73.66 0)
 			(effects
 				(font
@@
 		)
 		(property "Footprint" ""
-			(at 81.28 68.58 0)
+			(at 80.01 68.58 0)
 			(effects
 				(font
@@
 		)
 		(property "Datasheet" ""
-			(at 81.28 68.58 0)
+			(at 80.01 68.58 0)
 			(effects
 				(font
@@
 		)
 		(property "Description" "Power symbol creates a global label with name \"GND\" , ground"
-			(at 81.28 68.58 0)
+			(at 80.01 68.58 0)
 			(effects
 				(font
@@
 	(symbol
 		(lib_id "Device:L_Small")
-		(at 86.36 63.5 90)
+		(at 85.09 63.5 90)
 		(unit 1)
 		(exclude_from_sim no)
@@
 		(dnp no)
 		(property "Reference" "L7"
-			(at 86.36 58.42 90)
+			(at 85.09 58.42 90)
 			(effects
 				(font
@@
 		)
 		(property "Value" "5.1nH"
-			(at 86.36 60.96 90)
+			(at 85.09 60.96 90)
 			(effects
 				(font
@@
 		)
 		(property "Footprint" "Inductor_SMD:L_0402_1005Metric"
-			(at 86.36 63.5 0)
+			(at 85.09 63.5 0)
 			(effects
 				(font
@@
 		)
 		(property "Datasheet" "~"
-			(at 86.36 63.5 0)
+			(at 85.09 63.5 0)
 			(effects
 				(font
@@
 		)
 		(property "Description" "0603CS-5N1XJL"
-			(at 86.36 63.5 0)
+			(at 85.09 63.5 0)
 			(effects
 				(font
@@
 		)
 		(property "Manufacturer" "Coincraft"
-			(at 86.36 63.5 90)
+			(at 85.09 63.5 90)
 			(effects
 				(font
@@
 		)
 		(property "Part_Number" "0603CS-5N1XJLU"
-			(at 86.36 63.5 90)
-			(effects
-				(font
+			(at 85.09 63.5 90)
+			(effects
+				(font
