File: transceiver.kicad_sch (KiCad schematic)
At the start: 27 parts, among them J2 TagConnect_TC2030, U2 EFR32xG23xxxxF512xM48, Y1 32.768KHz, Y2 38.400MHz

Commit message: Readability updates
Parts:
- renumbered C5 to C1, C14 to C10, C15 to C11, C16 to C12, C17 to C13, C18 to C14, C19 to C15, C20 to C16, C21 to C17, C22 to C18, C6 to C2, C7 to C3, C8 to C4, C9 to C5, C10 to C6, C11 to C7, C12 to C8, C13 to C9, U2 to U1
Connections:
- net RF_IN renamed ANTENNA
Other:
- moved on the sheet: C14, C15, C16, L3, L4

Commit message: Routing updates
Parts:
- removed Y1: 32.768KHz, Oscillator:Oscillator_SMD_Abracon_ASCO-4Pin_1.6x1.2mm, symbol Oscillator:ASCO
- added Y3: 32.768KHz, Avionics_Feet:OSC_SIT1532AI-J4-DCC-32.768D, symbol Avionics_Symbols:SIT1532
- U1: value EFR32xG23xxxxF512xM48 -> EFR32FG23A010F256GM40; footprint Package_DFN_QFN:QFN-48-1EP_6x6mm_P0.4mm_EP4.3x4.3mm -> Package_DFN_QFN:QFN-40-1EP_5x5mm_P0.4mm_EP3.6x3.6mm; Information https://drzwave.blog/2022/07/21/z-wave-800-gpio-decoder-rin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 -> (none)
- Y2: value 38.400MHz -> 39MHz; footprint Oscillator:Oscillator_SMD_Abracon_ASCO-4Pin_1.6x1.2mm -> Crystal:Crystal_SMD_2016-4Pin_2.0x1.6mm
Connections:
- net +3V3: now also U1.32 (VREGVDD), U1.35 (AVDD), U1.36 (IOVDD), Y3.3 (VDD); no longer U1.38 (VREGVDD), U1.41 (AVDD), U1.42 (IOVDD)
- net CS: now also U1.4 (PC03); no longer U1.29 (PA04_TCLK)
- net GND: now also U1.13 (RFVSS), U1.33 (VREGVSS), U1.41 (PAD), Y3.1 (GND), Y3.4 (GND); no longer U1.15 (RFVSS), U1.39 (VREGVSS), U1.49 (PAD)
- net IN: now also U1.14 (SUBG_I1), U1.15 (SUBG_I0); no longer U1.16 (SUBG_I1), U1.17 (SUBG_I0)
- net MISO: now also U1.2 (PC01); no longer U1.32 (PA07_TD3)
- net MOSI: now also U1.6 (PC05); no longer U1.31 (PA06_TD2)
- net OUT: now also U1.16 (SUBG_O1), U1.17 (SUBG_O0); no longer U1.18 (SUBG_O1), U1.19 (SUBG_O0)
- net SCK: now also U1.8 (PC07); no longer U1.30 (PA05_TD1)
- net SWCLK: now also U1.22 (PA01_SWCLK); no longer U1.26 (PA01_SWCLK)
- net SWDIO: now also U1.23 (PA02_SWDIO); no longer U1.27 (PA02_SWDIO)
- net SWO: now also U1.24 (PA03_SWO); no longer U1.28 (PA03_SWO)
- net UART_RX: now also U1.26 (PA05); no longer U1.34 (PA09_URX)
- net UART_TX: now also U1.27 (PA06); no longer U1.33 (PA08_UTX)
- net VDCDC: now also U1.34 (DVDD); no longer U1.40 (DVDD)
- net VDDA: now also U1.12 (RFVDD), U1.18 (PAVDD); no longer U1.14 (RFVDD), U1.20 (PAVDD)
- net nRESET: now also U1.11 (nRESET); no longer U1.13 (~{RESET})
- net at Y2.3 (OUT): now also U1.9 (HFXTAL_I); no longer U1.11 (HFXTAL_I)
- net PC02: now reaches U1.3 (PC02)
- net at C18.1: now also U1.30 (DECOUPLE); no longer U1.36 (DECOUPLE)
- net at L4.2: now also U1.31 (VREGSW); no longer U1.37 (VREGSW)
- removed net PD04: U1.44 (PD04_PDATA)
- new net: U1.39 (PD01_LFXI), Y3.2 (OUT)
- no-connect marks 20 -> 12
Other:
- moved on the sheet: C16, C17, C18, J2, L3, L4, Y2
